File: hardware/LoRa.kicad_sch (KiCad schematic)
At the start: 32 parts, among them J2 Conn_Coaxial, U8 SX1261IMLTRT, U9 4259-63, Y1 Crystal_GND3

Commit message: Finished Schematic and Routed PCB
Connections:
- net GND: now also U8.20 (GND)
- net DIO1: now reaches U8.13 (DIO1)
- net BUSY: now reaches U8.14 (BUSY)
- net NRESET: now reaches U8.15 (NRESET)
- net MISO: now reaches U8.16 (MISO)
- net MOSI: now reaches U8.17 (MOSI)
- net SCK: now reaches U8.18 (SCK)
- net NSS: now reaches U8.19 (NSS)
Changed lines of the file:
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@@
 		)
 	)
-	(global_label "DIO3"
-		(shape input)
-		(at 73.66 67.31 180)
-		(fields_autoplaced yes)
+	(label "DIO2"
+		(at 212.09 118.11 180)
 		(effects
 			(font
 				(size 1.27 1.27)
 			)
-			(justify right)
-		)
-		(property "Intersheetrefs" "${INTERSHEET_REFS}"
-			(at 66.26 67.31 0)
-			(effects
-				(font
-					(size 1.27 1.27)
-				)
-				(justify right)
-				(hide yes)
-			)
-		)
-	)
-	(global_label "DIO2"
-		(shape input)
+			(justify right bottom)
+		)
+	)
+	(label "DIO2"
 		(at 82.55 82.55 180)
-		(fields_autoplaced yes)
 		(effects
 			(font
 				(size 1.27 1.27)
 			)
-			(justify right)
-		)
-		(property "Intersheetrefs" "${INTERSHEET_REFS}"
-			(at 75.15 82.55 0)
-			(effects
-				(font
-					(size 1.27 1.27)
-				)
-				(justify right)
-				(hide yes)
-			)
+			(justify right bottom)
 		)
 	)
@@
 		)
 	)
-	(global_label "VDD_RADIO"
+	(hierarchical_label "DIO3"
 		(shape input)
-		(at 55.88 85.09 180)
-		(fields_autoplaced yes)
+		(at 73.66 67.31 180)
 		(effects
 			(font
@@
 			(justify right)
 		)
-		(property "Intersheetrefs" "${INTERSHEET_REFS}"
-			(at 42.7347 85.09 0)
-			(effects
-				(font
-					(size 1.27 1.27)
-				)
-				(justify right)
-				(hide yes)
-			)
-		)
-	)
-	(global_label "DIO2"
+	)
+	(hierarchical_label "MISO"
 		(shape input)
-		(at 212.09 118.11 180)
-		(fields_autoplaced yes)
+		(at 133.35 77.47 0)
 		(effects
 			(font
 				(size 1.27 1.27)
 			)
+			(justify left)
+		)
+	)
+	(hierarchical_label "SCK"
+		(shape input)
+		(at 133.35 72.39 0)
+		(effects
+			(font
+				(size 1.27 1.27)
+			)
+			(justify left)
+		)
+	)
+	(hierarchical_label "NSS"
+		(shape input)
+		(at 133.35 69.85 0)
+		(effects
+			(font
+				(size 1.27 1.27)
+			)
+			(justify left)
+		)
+	)
+	(hierarchical_label "DIO1"
+		(shape input)
+		(at 133.35 85.09 0)
+		(effects
+			(font
+				(size 1.27 1.27)
+			)
+			(justify left)
+		)
+	)
+	(hierarchical_label "MOSI"
+		(shape input)
+		(at 133.35 74.93 0)
+		(effects
+			(font
+				(size 1.27 1.27)
+			)
+			(justify left)
+		)
+	)
+	(hierarchical_label "BUSY"
+		(shape input)
+		(at 133.35 82.55 0)
+		(effects
+			(font
+				(size 1.27 1.27)
+			)
+			(justify left)
+		)
+	)
+	(hierarchical_label "VDD_RADIO"
+		(shape input)
+		(at 55.88 85.09 180)
+		(effects
+			(font
+				(size 1.27 1.27)
+			)
 			(justify right)
 		)
-		(property "Intersheetrefs" "${INTERSHEET_REFS}"
-			(at 204.69 118.11 0)
-			(effects
-				(font
-					(size 1.27 1.27)
-				)
-				(justify right)
-				(hide yes)
-			)
+	)
+	(hierarchical_label "NRESET"
+		(shape input)
+		(at 133.35 80.01 0)
+		(effects
+			(font
+				(size 1.27 1.27)
+			)
+			(justify left)
 		)
 	)
@@
 					(unit 1)
 				)
+			)
+		)
+	)
+	(symbol
+		(lib_id "power:GND")
+		(at 133.35 67.31 90)
+		(unit 1)
+		(exclude_from_sim no)
+		(in_bom yes)
+		(on_board yes)
+		(dnp no)
+		(property "Reference" "#PWR033"
+			(at 139.7 67.31 0)
+			(effects
+				(font
+					(size 1.27 1.27)
+				)
+				(hide yes)
+			)
+		)
+		(property "Value" "GND"
+			(at 136.906 67.31 90)
+			(effects
+				(font
+					(size 1.27 1.27)
+				)
+				(justify right)
+			)
+		)
+		(property "Footprint" ""
+			(at 133.35 67.31 0)
+			(effects
+				(font
+					(size 1.27 1.27)
+				)
+				(hide yes)
+			)
+		)
+		(property "Datasheet" ""
+			(at 133.35 67.31 0)
+			(effects
+				(font
+					(size 1.27 1.27)
+				)
+				(hide yes)
+			)
+		)
+		(property "Description" "Power symbol creates a global label with name \"GND\" , ground"
+			(at 133.35 67.31 0)
+			(effects
+				(font
+					(size 1.27 1.27)
+				)
+				(hide yes)
+			)
+		)
+		(pin "1"
+		)
+		(instances
+			(project "teachtaire"
+				(path "/43b606e0-d389-434f-90f5-9db489b60c46/243b3313-f54d-44cb-8514-68b2127144cd"
+					(reference "#PWR033")
+					(unit 1)
+				)
