File: hardware/power.kicad_sch (KiCad schematic)
At the start: 22 parts, among them U4 MPM3650CGQW-P, U9 TLV75533PDRV

Commit message: fixed the fuck-ups
Parts:
- gave numbers to parts that had none: 10
- renumbered C3 to C24, C4 to C25, C5 to C30, C6 to C31, C7 to C34, C8 to C35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
