File: hardware/teachtaire.kicad_sch (KiCad schematic)
At the start: 42 parts, among them J1 39-29-1048, J2 ESQ-110-X-X-D, J3 Conn_Coaxial, J4 5023860570, Q1 NMOS, Q2 IPD90P04P4L04ATMA1, U1 MAX-M10S, U2 STM32F072C8Tx, U3 TJA1051T/3/1J, U4 RF-LORA-868-SO

Commit message: ready for review the twost
Parts:
- added 3V3D1, 3V3RF1, CAN+1, CAN-1, LD0, LD1, LD2, LD3, LD4, LD5, VIN1: S2761-46R, HARWIN_S2761-46R, symbol S2761-46R:S2761-46R
- renumbered D4 to D1, D1 to D2, D2 to D3, D3 to D4
Connections:
- net +3V3D: now also 3V3D1.1
- net +3V3RF: now also 3V3RF1.1
- net CANo_+: now also CAN+1.1
- net CANo_-: now also CAN-1.1
- net LoRa_DIO0: now also LD0.1
- net LoRa_DIO1: now also LD1.1
- net LoRa_DIO2: now also LD2.1
- net LoRa_DIO3: now also LD3.1
- net LoRa_DIO4: now also LD4.1
- net LoRa_DIO5: now also LD5.1
- net VBAT: now also VIN1.1
