File: hardware/GNSS.kicad_sch (KiCad schematic)
At the start: 14 parts, among them J1 Conn_Coaxial, Q1 PMOS, Q2 NMOS, U5 LT6003HDC-TRMPBF, U6 NC7WZ07P6X, U7 NC7WZ07P6X

Commit message: Added values to components
Parts:
- C1: value C -> 47pF
- C2: value C -> 10nF
- L1: value L -> 27nH
- R2: value R -> 10Ω
- R3, R5: value R -> 100kΩ
- R4: value R -> 560Ω
Changed lines of the file:
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@@
 			)
 		)
-		(property "Value" "C"
+		(property "Value" "47pF"
 			(at 62.23 36.83 90)
 			(effects
@@
 			)
 		)
-		(property "Value" "R"
+		(property "Value" "560Ω"
 			(at 63.5 123.1899 0)
 			(effects
@@
 			)
 		)
-		(property "Value" "R"
+		(property "Value" "10Ω"
 			(at 46.99 66.0399 0)
 			(effects
@@
 			)
 		)
-		(property "Value" "C"
+		(property "Value" "10nF"
 			(at 59.69 50.8 90)
 			(effects
@@
 			)
 		)
-		(property "Value" "R"
+		(property "Value" "100kΩ"
 			(at 63.5 133.3499 0)
 			(effects
@@
 			)
 		)
-		(property "Value" "L"
+		(property "Value" "27nH"
 			(at 45.72 52.0699 0)
 			(effects
@@
 			)
 		)
-		(property "Value" "R"
+		(property "Value" "100kΩ"
 			(at 50.8 82.55 90)
 			(effects

Commit message: Finished Schematic and Routed PCB
Parts:
- C1, C2, FB1: footprint (none) -> Capacitor_SMD:C_0402_1005Metric
- J1: footprint (none) -> Connector_Coaxial:U.FL_Molex_MCRF_73412-0110_Vertical
- L1: footprint (none) -> Inductor_SMD:L_0402_1005Metric
- Q1, Q2: footprint (none) -> Package_TO_SOT_SMD:SOT-23
- R2, R3, R4, R5: footprint (none) -> Resistor_SMD:R_0402_1005Metric
- U6, U7: footprint SC-88/SC70-6/SOT-363_419B-02_ONS -> SC-88&slash_SC70-6&slash_SOT-363_419B-02_ONS
Connections:
- net antenna supply renamed Antenna Supply
Changed lines of the file:
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@@
 		)
 	)
-	(global_label "ANT_DETECT"
+	(hierarchical_label "ANT_SHORT_N"
 		(shape input)
-		(at 161.29 129.54 0)
-		(fields_autoplaced yes)
+		(at 156.21 152.4 0)
 		(effects
 			(font
@@
 			(justify left)
 		)
-		(property "Intersheetrefs" "${INTERSHEET_REFS}"
-			(at 175.4027 129.54 0)
-			(effects
-				(font
-					(size 1.27 1.27)
-				)
-				(justify left)
-				(hide yes)
-			)
-		)
-	)
-	(global_label "RF_IN"
+	)
+	(hierarchical_label "RF_IN"
 		(shape input)
 		(at 80.01 41.91 0)
-		(fields_autoplaced yes)
 		(effects
 			(font
@@
 			(justify left)
 		)
-		(property "Intersheetrefs" "${INTERSHEET_REFS}"
-			(at 88.2567 41.91 0)
-			(effects
-				(font
-					(size 1.27 1.27)
-				)
-				(justify left)
-				(hide yes)
-			)
-		)
-	)
-	(global_label "ANT_SHORT_N"
+	)
+	(hierarchical_label "Antenna Supply"
 		(shape input)
-		(at 156.21 152.4 0)
-		(fields_autoplaced yes)
+		(at 44.45 95.25 270)
 		(effects
 			(font
 				(size 1.27 1.27)
 			)
-			(justify left)
-		)
-		(property "Intersheetrefs" "${INTERSHEET_REFS}"
-			(at 171.9557 152.4 0)
-			(effects
-				(font
-					(size 1.27 1.27)
-				)
-				(justify left)
-				(hide yes)
-			)
-		)
-	)
-	(global_label "ANT_OFF_N"
+			(justify right)
+		)
+	)
+	(hierarchical_label "ANT_DETECT"
 		(shape input)
-		(at 85.09 90.17 0)
-		(fields_autoplaced yes)
+		(at 161.29 129.54 0)
 		(effects
 			(font
@@
 			(justify left)
 		)
-		(property "Intersheetrefs" "${INTERSHEET_REFS}"
-			(at 98.2353 90.17 0)
-			(effects
-				(font
-					(size 1.27 1.27)
-				)
-				(justify left)
-				(hide yes)
-			)
-		)
-	)
-	(global_label "V_ANT"
+	)
+	(hierarchical_label "ANT_OFF_N"
 		(shape input)
-		(at 161.29 133.35 0)
-		(fields_autoplaced yes)
+		(at 85.09 90.17 0)
 		(effects
 			(font
@@
 			(justify left)
 		)
-		(property "Intersheetrefs" "${INTERSHEET_REFS}"
-			(at 169.7181 133.35 0)
-			(effects
-				(font
-					(size 1.27 1.27)
-				)
-				(justify left)
-				(hide yes)
-			)
-		)
-	)
-	(global_label "V_ANT"
+	)
+	(hierarchical_label "V_ANT"
 		(shape input)
-		(at 115.57 121.92 90)
-		(fields_autoplaced yes)
+		(at 161.29 133.35 0)
 		(effects
 			(font
@@
 			(justify left)
 		)
-		(property "Intersheetrefs" "${INTERSHEET_REFS}"
-			(at 115.57 113.4919 90)
-			(effects
-				(font
-					(size 1.27 1.27)
-				)
-				(justify left)
-				(hide yes)
-			)
-		)
-	)
-	(global_label "V_ANT"
+	)
+	(hierarchical_label "V_ANT"
 		(shape input)
-		(at 158.75 156.21 0)
-		(fields_autoplaced yes)
+		(at 115.57 121.92 90)
 		(effects
 			(font
@@
 			(justify left)
 		)
-		(property "Intersheetrefs" "${INTERSHEET_REFS}"
-			(at 167.1781 156.21 0)
-			(effects
-				(font
-					(size 1.27 1.27)
-				)
-				(justify left)
-				(hide yes)
-			)
-		)
-	)
-	(global_label "antenna supply"
+	)
+	(hierarchical_label "V_ANT"
 		(shape input)
-		(at 44.45 95.25 270)
-		(fields_autoplaced yes)
+		(at 158.75 156.21 0)
 		(effects
 			(font
 				(size 1.27 1.27)
 			)
-			(justify right)
-		)
-		(property "Intersheetrefs" "${INTERSHEET_REFS}"
-			(at 44.45 112.87 90)
-			(effects
-				(font
-					(size 1.27 1.27)
-				)
-				(justify right)
-				(hide yes)
-			)
+			(justify left)
 		)
 	)
@@
 			)
 		)
-		(property "Footprint" ""
+		(property "Footprint" "Capacitor_SMD:C_0402_1005Metric"
 			(at 66.04 40.9448 0)
 			(effects
@@
 			)
 		)
-		(property "Footprint" ""
+		(property "Footprint" "Resistor_SMD:R_0402_1005Metric"
 			(at 59.182 121.92 90)
 			(effects
@@
 			)
 		)
-		(property "Footprint" ""
+		(property "Footprint" "Resistor_SMD:R_0402_1005Metric"
 			(at 42.672 64.77 90)
 			(effects
@@
 			)
 		)
-		(property "Footprint" ""
+		(property "Footprint" "Package_TO_SOT_SMD:SOT-23"
 			(at 67.31 92.71 0)
 			(effects
@@
 			)
 		)
-		(property "Footprint" ""
+		(property "Footprint" "Package_TO_SOT_SMD:SOT-23"
 			(at 41.91 81.28 0)
 			(effects
@@
 			)
 		)
-		(property "Footprint" ""
+		(property "Footprint" "Capacitor_SMD:C_0402_1005Metric"
 			(at 63.5 54.9148 0)
 			(effects
@@
 			)
 		)
-		(property "Footprint" ""
+		(property "Footprint" "Resistor_SMD:R_0402_1005Metric"
 			(at 59.182 132.08 90)
 			(effects
@@
 			)
 		)
-		(property "Footprint" ""
+		(property "Footprint" "Inductor_SMD:L_0402_1005Metric"
 			(at 44.45 50.8 0)
 			(effects
@@
 			)
 		)
-		(property "Footprint" "SC-88/SC70-6/SOT-363_419B-02_ONS"
+		(property "Footprint" "SC-88&slash_SC70-6&slash_SOT-363_419B-02_ONS"
 			(at 115.57 152.4 0)
 			(effects
@@
 			)
 		)
-		(property "Footprint" "SC-88/SC70-6/SOT-363_419B-02_ONS"
+		(property "Footprint" "SC-88&slash_SC70-6&slash_SOT-363_419B-02_ONS"
 			(at 115.57 129.54 0)
 			(effects
@@
 			)
 		)
-		(property "Footprint" ""
+		(property "Footprint" "Capacitor_SMD:C_0402_1005Metric"
 			(at 76.2 40.132 90)
 			(effects
@@
 			)
 		)
-		(property "Footprint" ""
+		(property "Footprint" "Resistor_SMD:R_0402_1005Metric"
 			(at 50.8 88.138 90)
 			(effects
@@
 			)
 		)
-		(property "Footprint" ""
+		(property "Footprint" "Connector_Coaxial:U.FL_Molex_MCRF_73412-0110_Vertical"
 			(at 44.45 27.94 0)
 			(effects

Commit message: Changes from Reddit review 1
Changed connector, impedance matched the RF traces, changed board to square
Parts:
- J1: footprint Connector_Coaxial:U.FL_Molex_MCRF_73412-0110_Vertical -> Connector_Coaxial:SMA_BAT_Wireless_BWSMA-KWE-Z001
Changed lines of the file:
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@@
 			)
 		)
-		(property "Footprint" "Connector_Coaxial:U.FL_Molex_MCRF_73412-0110_Vertical"
+		(property "Footprint" "Connector_Coaxial:SMA_BAT_Wireless_BWSMA-KWE-Z001"
 			(at 44.45 27.94 0)
 			(effects

Commit message: many fatal fuck-ups found
Parts:
- removed FB1: FerriteBead, Capacitor_SMD:C_0402_1005Metric, symbol Device:FerriteBead
- added R14, R15: 0Ω, Resistor_SMD:R_0402_1005Metric, symbol Device:R
Connections:
- net ANT_DETECT: now also R14.2; no longer U6.6 (Y1)
- net ANT_SHORT_N: now also R15.2; no longer U7.6 (Y1)
- net Antenna Supply: now also Q1.3 (S); no longer Q1.1 (D)
- net GND: now also Q2.3 (S); no longer Q2.1 (D)
- net RF_IN: now also C1.2
- net at R2.2, R4.1: now also Q1.1 (D); no longer Q1.3 (S)
- net at Q1.2 (G), R3.2: now also Q2.1 (D); no longer Q2.3 (S)
- net V_ANT renamed +3V3D
- new net: R15.1, U7.6 (Y1)
- new net: R14.1, U6.6 (Y1)
Other:
- moved on the sheet: C1, L1, Q1, Q2, R2, R3, R4, R5, U5, U6, U7

Commit message: fixed the fuck-ups
Parts:
- renumbered C1 to C21, C2 to C22, J1 to J5, Q1 to Q3, Q2 to Q4, R14 to R10, R15 to R11, R2 to R6, R3 to R7, R4 to R8, R5 to R9
Changed lines of the file:
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@@
 		(dnp no)
 		(fields_autoplaced yes)
-		(property "Reference" "#PWR09"
+		(property "Reference" "#PWR044"
 			(at 69.85 113.03 0)
 			(effects
@@
 			(project "teachtaire"
 				(path "/43b606e0-d389-434f-90f5-9db489b60c46/a8c66ae0-f2ee-422a-8d95-b403d0fcd214"
-					(reference "#PWR09")
+					(reference "#PWR044")
 					(unit 1)
 				)
@@
 		(dnp no)
 		(fields_autoplaced yes)
-		(property "Reference" "C1"
+		(property "Reference" "C21"
 			(at 59.69 34.29 90)
 			(effects
@@
 			(project "teachtaire"
 				(path "/43b606e0-d389-434f-90f5-9db489b60c46/a8c66ae0-f2ee-422a-8d95-b403d0fcd214"
-					(reference "C1")
+					(reference "C21")
 					(unit 1)
 				)
@@
 		(dnp no)
 		(fields_autoplaced yes)
-		(property "Reference" "R4"
+		(property "Reference" "R8"
 			(at 63.5 128.2699 0)
 			(effects
@@
 			(project "teachtaire"
 				(path "/43b606e0-d389-434f-90f5-9db489b60c46/a8c66ae0-f2ee-422a-8d95-b403d0fcd214"
-					(reference "R4")
+					(reference "R8")
 					(unit 1)
 				)
@@
 		(dnp no)
 		(fields_autoplaced yes)
-		(property "Reference" "R2"
+		(property "Reference" "R6"
 			(at 46.99 74.9299 0)
 			(effects
@@
 			(project "teachtaire"
 				(path "/43b606e0-d389-434f-90f5-9db489b60c46/a8c66ae0-f2ee-422a-8d95-b403d0fcd214"
-					(reference "R2")
+					(reference "R6")
 					(unit 1)
 				)
@@
 		(on_board yes)
 		(dnp no)
-		(property "Reference" "Q2"
+		(property "Reference" "Q4"
 			(at 67.056 100.584 0)
 			(effects
@@
 			(project "teachtaire"
 				(path "/43b606e0-d389-434f-90f5-9db489b60c46/a8c66ae0-f2ee-422a-8d95-b403d0fcd214"
-					(reference "Q2")
+					(reference "Q4")
 					(unit 1)
 				)
@@
 		(on_board yes)
 		(dnp no)
-		(property "Reference" "Q1"
+		(property "Reference" "Q3"
 			(at 41.91 91.44 0)
 			(effects
@@
 			(project "teachtaire"
 				(path "/43b606e0-d389-434f-90f5-9db489b60c46/a8c66ae0-f2ee-422a-8d95-b403d0fcd214"
-					(reference "Q1")
+					(reference "Q3")
 					(unit 1)
 				)
@@
 		(dnp no)
 		(fields_autoplaced yes)
-		(property "Reference" "C2"
+		(property "Reference" "C22"
 			(at 59.69 48.26 90)
 			(effects
@@
 			(project "teachtaire"
 				(path "/43b606e0-d389-434f-90f5-9db489b60c46/a8c66ae0-f2ee-422a-8d95-b403d0fcd214"
-					(reference "C2")
+					(reference "C22")
 					(unit 1)
 				)
@@
 		(dnp no)
 		(fields_autoplaced yes)
-		(property "Reference" "#PWR010"
+		(property "Reference" "#PWR042"
 			(at 60.96 149.86 0)
 			(effects
@@
 			(project "teachtaire"
 				(path "/43b606e0-d389-434f-90f5-9db489b60c46/a8c66ae0-f2ee-422a-8d95-b403d0fcd214"
-					(reference "#PWR010")
+					(reference "#PWR042")
 					(unit 1)
 				)
@@
 		(dnp no)
 		(fields_autoplaced yes)
-		(property "Reference" "#PWR024"
+		(property "Reference" "#PWR048"
 			(at 153.67 162.56 0)
 			(effects
@@
 			(project "teachtaire"
 				(path "/43b606e0-d389-434f-90f5-9db489b60c46/a8c66ae0-f2ee-422a-8d95-b403d0fcd214"
-					(reference "#PWR024")
+					(reference "#PWR048")
 					(unit 1)
 				)
@@
 		(on_board yes)
 		(dnp no)
-		(property "Reference" "#PWR012"
+		(property "Reference" "#PWR047"
 			(at 115.57 172.72 0)
 			(effects
@@
 			(project "teachtaire"
 				(path "/43b606e0-d389-434f-90f5-9db489b60c46/a8c66ae0-f2ee-422a-8d95-b403d0fcd214"
-					(reference "#PWR012")
+					(reference "#PWR047")
 					(unit 1)
 				)
@@
 		(dnp no)
 		(fields_autoplaced yes)
-		(property "Reference" "#PWR025"
+		(property "Reference" "#PWR049"
 			(at 156.21 139.7 0)
 			(effects
@@
 			(project "teachtaire"
 				(path "/43b606e0-d389-434f-90f5-9db489b60c46/a8c66ae0-f2ee-422a-8d95-b403d0fcd214"
-					(reference "#PWR025")
+					(reference "#PWR049")
 					(unit 1)
 				)
@@
 		(dnp no)
 		(fields_autoplaced yes)
-		(property "Reference" "#PWR01"
+		(property "Reference" "#PWR041"
 			(at 55.88 27.94 0)
 			(effects
@@
 			(project "teachtaire"
 				(path "/43b606e0-d389-434f-90f5-9db489b60c46/a8c66ae0-f2ee-422a-8d95-b403d0fcd214"
-					(reference "#PWR01")
+					(reference "#PWR041")
 					(unit 1)
 				)
@@
 		(on_board yes)
 		(dnp no)
-		(property "Reference" "#PWR011"
+		(property "Reference" "#PWR046"
 			(at 115.57 149.86 0)
 			(effects
@@
 			(project "teachtaire"
 				(path "/43b606e0-d389-434f-90f5-9db489b60c46/a8c66ae0-f2ee-422a-8d95-b403d0fcd214"
-					(reference "#PWR011")
+					(reference "#PWR046")
 					(unit 1)
 				)
@@
 		(dnp no)
 		(fields_autoplaced yes)
-		(property "Reference" "R5"
+		(property "Reference" "R9"
 			(at 63.5 138.4299 0)
 			(effects
@@
 			(project "teachtaire"
 				(path "/43b606e0-d389-434f-90f5-9db489b60c46/a8c66ae0-f2ee-422a-8d95-b403d0fcd214"
-					(reference "R5")
+					(reference "R9")
 					(unit 1)
 				)
@@
 		(on_board yes)
 		(dnp no)
-		(property "Reference" "#PWR026"
+		(property "Reference" "#PWR045"
 			(at 111.76 134.62 0)
 			(effects
@@
 			(project "teachtaire"
 				(path "/43b606e0-d389-434f-90f5-9db489b60c46/a8c66ae0-f2ee-422a-8d95-b403d0fcd214"
-					(reference "#PWR026")
+					(reference "#PWR045")
 					(unit 1)
 				)
@@
 		(dnp no)
 		(fields_autoplaced yes)
-		(property "Reference" "R14"
+		(property "Reference" "R10"
 			(at 161.29 130.81 90)
 			(effects
@@
 			(project "teachtaire"
 				(path "/43b606e0-d389-434f-90f5-9db489b60c46/a8c66ae0-f2ee-422a-8d95-b403d0fcd214"
-					(reference "R14")
+					(reference "R10")
 					(unit 1)
 				)
@@
 		(on_board yes)
 		(dnp no)
-		(property "Reference" "R3"
+		(property "Reference" "R7"
 			(at 50.8 92.964 90)
 			(effects
@@
 			(project "teachtaire"
 				(path "/43b606e0-d389-434f-90f5-9db489b60c46/a8c66ae0-f2ee-422a-8d95-b403d0fcd214"
-					(reference "R3")
+					(reference "R7")
 					(unit 1)
 				)
@@
 		(dnp no)
 		(fields_autoplaced yes)
-		(property "Reference" "#PWR08"
+		(property "Reference" "#PWR043"
 			(at 69.85 55.88 0)
 			(effects
@@
 			(project "teachtaire"
 				(path "/43b606e0-d389-434f-90f5-9db489b60c46/a8c66ae0-f2ee-422a-8d95-b403d0fcd214"
-					(reference "#PWR08")
+					(reference "#PWR043")
 					(unit 1)
 				)
@@
 		(dnp no)
 		(fields_autoplaced yes)
-		(property "Reference" "J1"
+		(property "Reference" "J5"
 			(at 44.7432 21.59 90)
 			(effects
@@
 			(project "teachtaire"
 				(path "/43b606e0-d389-434f-90f5-9db489b60c46/a8c66ae0-f2ee-422a-8d95-b403d0fcd214"
-					(reference "J1")
+					(reference "J5")
 					(unit 1)
 				)
@@
 		(dnp no)
 		(fields_autoplaced yes)
-		(property "Reference" "R15"
+		(property "Reference" "R11"
 			(at 161.29 153.67 90)
 			(effects
@@
 			(project "teachtaire"
 				(path "/43b606e0-d389-434f-90f5-9db489b60c46/a8c66ae0-f2ee-422a-8d95-b403d0fcd214"
-					(reference "R15")
-					(unit 1)
-				)
+					(reference "R11")
+					(unit 1)
+				)

Commit message: crimes
Parts:
- removed J5: Conn_Coaxial, Connector_Coaxial:SMA_BAT_Wireless_BWSMA-KWE-Z001, symbol Connector:Conn_Coaxial
- added J6: U.FL-R-SMT-1_10_, HRS_U.FL-R-SMT-1_10_, symbol U.FL-R-SMT-1_10_:U.FL-R-SMT-1_10_
Connections:
- net GND: now also J6.1, J6.3
- net at C21.1, L1.1: now also J6.2
Changed lines of the file:
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@@
 	(wire
 		(pts
-			(xy 44.45 41.91) (xy 44.45 33.02)
+			(xy 44.45 30.48) (xy 44.45 41.91)
 		)
 		(stroke
@@
 	)
 	(symbol
+		(lib_id "U.FL-R-SMT-1_10_:U.FL-R-SMT-1_10_")
+		(at 44.45 27.94 90)
+		(unit 1)
+		(exclude_from_sim no)
+		(in_bom yes)
+		(on_board yes)
+		(dnp no)
+		(property "Reference" "J6"
+			(at 43.434 25.908 0)
+			(effects
+				(font
+					(size 1.27 1.27)
+				)
+				(justify left)
+			)
+		)
+		(property "Value" "U.FL-R-SMT-1_10_"
+			(at 66.04 25.146 90)
+			(effects
+				(font
+					(size 1.27 1.27)
+				)
+				(justify left)
+			)
+		)
+		(property "Footprint" "HRS_U.FL-R-SMT-1_10_"
+			(at 44.45 27.94 0)
+			(effects
+				(font
+					(size 1.27 1.27)
+				)
+				(justify bottom)
+				(hide yes)
+			)
+		)
+		(property "Datasheet" ""
+			(at 44.45 27.94 0)
+			(effects
+				(font
+					(size 1.27 1.27)
+				)
+				(hide yes)
+			)
+		)
+		(property "Description" ""
+			(at 44.45 27.94 0)
+			(effects
+				(font
+					(size 1.27 1.27)
+				)
+				(hide yes)
+			)
+		)
+		(property "MF" "Hirose"
+			(at 44.45 27.94 0)
+			(effects
+				(font
+					(size 1.27 1.27)
+				)
+				(justify bottom)
+				(hide yes)
+			)
+		)
+		(property "DESCRIPTION" "U.FL Series 6 Ghz 50 Ohm Ultra-small SMT Coaxial Cable Receptacle"
+			(at 44.45 27.94 0)
+			(effects
+				(font
+					(size 1.27 1.27)
+				)
+				(justify bottom)
+				(hide yes)
+			)
+		)
+		(property "PACKAGE" "None"
+			(at 44.45 27.94 0)
+			(effects
+				(font
+					(size 1.27 1.27)
+				)
+				(justify bottom)
+				(hide yes)
+			)
+		)
+		(property "PRICE" "0.71 USD"
+			(at 44.45 27.94 0)
+			(effects
+				(font
+					(size 1.27 1.27)
+				)
+				(justify bottom)
+				(hide yes)
+			)
+		)
+		(property "Package" "None"
+			(at 44.45 27.94 0)
+			(effects
+				(font
+					(size 1.27 1.27)
+				)
+				(justify bottom)
+				(hide yes)
+			)
+		)
+		(property "Check_prices" "https://www.snapeda.com/parts/U.FL-R-SMT-1(10)/Hirose+Electric+Co+Ltd/view-part/?ref=eda"
+			(at 44.45 27.94 0)
+			(effects
+				(font
+					(size 1.27 1.27)
+				)
+				(justify bottom)
+				(hide yes)
+			)
+		)
+		(property "STANDARD" "Manufacturer Recommendation"
+			(at 44.45 27.94 0)
+			(effects
+				(font
+					(size 1.27 1.27)
+				)
+				(justify bottom)
+				(hide yes)
+			)
+		)
+		(property "SnapEDA_Link" "https://www.snapeda.com/parts/U.FL-R-SMT-1(10)/Hirose+Electric+Co+Ltd/view-part/?ref=snap"
+			(at 44.45 27.94 0)
+			(effects
+				(font
+					(size 1.27 1.27)
+				)
+				(justify bottom)
+				(hide yes)
+			)
+		)
+		(property "MP" "U.FL-R-SMT-1(10)"
+			(at 44.45 27.94 0)
+			(effects
+				(font
+					(size 1.27 1.27)
+				)
+				(justify bottom)
+				(hide yes)
+			)
+		)
+		(property "Price" "None"
+			(at 44.45 27.94 0)
+			(effects
+				(font
+					(size 1.27 1.27)
+				)
+				(justify bottom)
+				(hide yes)
+			)
+		)
+		(property "Description_1" "U.FL (UMCC) Connector Receptacle, Male Pin 50 Ohms Surface Mount Solder"
+			(at 44.45 27.94 0)
+			(effects
+				(font
+					(size 1.27 1.27)
+				)
+				(justify bottom)
+				(hide yes)
+			)
+		)
+		(property "Availability" "In Stock"
+			(at 44.45 27.94 0)
+			(effects
+				(font
+					(size 1.27 1.27)
+				)
+				(justify bottom)
+				(hide yes)
+			)
+		)
+		(property "AVAILABILITY" "Good"
+			(at 44.45 27.94 0)
+			(effects
+				(font
+					(size 1.27 1.27)
+				)
+				(justify bottom)
+				(hide yes)
+			)
+		)
+		(property "MANUFACTURER" "Hirose"
+			(at 44.45 27.94 0)
+			(effects
+				(font
+					(size 1.27 1.27)
+				)
+				(justify bottom)
+				(hide yes)
+			)
+		)
+		(pin "1"
+		)
+		(pin "2"
+		)
+		(pin "3"
+		)
+		(instances
+			(project "teachtaire"
+				(path "/43b606e0-d389-434f-90f5-9db489b60c46/a8c66ae0-f2ee-422a-8d95-b403d0fcd214"
+					(reference "J6")
+					(unit 1)
+				)
+			)
+		)
+	)
+	(symbol
 		(lib_id "power:GND")
 		(at 60.96 143.51 0)
@@
 	(symbol
 		(lib_id "power:GND")
-		(at 49.53 27.94 90)
+		(at 46.99 30.48 90)
 		(unit 1)
 		(exclude_from_sim no)
@@
 		(fields_autoplaced yes)
 		(property "Reference" "#PWR041"
-			(at 55.88 27.94 0)
+			(at 53.34 30.48 0)
 			(effects
 				(font
@@
 		)
 		(property "Value" "GND"
-			(at 53.34 27.9399 90)
+			(at 50.8 30.4799 90)
 			(effects
 				(font
@@
 		)
 		(property "Footprint" ""
-			(at 49.53 27.94 0)
+			(at 46.99 30.48 0)
 			(effects
 				(font
@@
 		)
 		(property "Datasheet" ""
-			(at 49.53 27.94 0)
+			(at 46.99 30.48 0)
 			(effects
 				(font
@@
 		)
 		(property "Description" "Power symbol creates a global label with name \"GND\" , ground"
-			(at 49.53 27.94 0)
+			(at 46.99 30.48 0)
 			(effects
 				(font
@@
 					(unit 1)
 				)
-			)
-		)
-	)
-	(symbol
-		(lib_id "Connector:Conn_Coaxial")
-		(at 44.45 27.94 90)
-		(unit 1)
-		(exclude_from_sim no)
-		(in_bom yes)
-		(on_board yes)
-		(dnp no)
-		(fields_autoplaced yes)
-		(property "Reference" "J5"
-			(at 44.7432 21.59 90)
-			(effects
-				(font
-					(size 1.27 1.27)
-				)
-			)
-		)
-		(property "Value" "Conn_Coaxial"
-			(at 44.7432 24.13 90)
-			(effects
-				(font
-					(size 1.27 1.27)
-				)
-			)
-		)
-		(property "Footprint" "Connector_Coaxial:SMA_BAT_Wireless_BWSMA-KWE-Z001"
-			(at 44.45 27.94 0)
-			(effects
-				(font
-					(size 1.27 1.27)
-				)
-				(hide yes)
-			)
-		)
-		(property "Datasheet" "~"
-			(at 44.45 27.94 0)
-			(effects
-				(font
-					(size 1.27 1.27)
-				)
-				(hide yes)
-			)
-		)
-		(property "Description" "coaxial connector (BNC, SMA, SMB, SMC, Cinch/RCA, LEMO, ...)"
-			(at 44.45 27.94 0)
-			(effects
-				(font
-					(size 1.27 1.27)
-				)
-				(hide yes)
-			)
-		)
-		(pin "2"
-		)
-		(pin "1"
-		)
-		(instances
-			(project "teachtaire"
-				(path "/43b606e0-d389-434f-90f5-9db489b60c46/a8c66ae0-f2ee-422a-8d95-b403d0fcd214"
-					(reference "J5")
-					(unit 1)
-				)
