File: hardware/GNSS.kicad_sch (KiCad schematic)
At the start: 15 parts, among them J6 U.FL-R-SMT-1_10_, Q3 PMOS, Q4 NMOS, U5 LT6003HDC-TRMPBF, U6 NC7WZ07P6X, U7 NC7WZ07P6X

Commit message: hardware done
Parts:
- C22: footprint Capacitor_SMD:C_0402_1005Metric -> Capacitor_SMD:C_0603_1608Metric
Changed lines of the file:
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@@
 			)
 		)
-		(property "Footprint" "Capacitor_SMD:C_0402_1005Metric"
+		(property "Footprint" "Capacitor_SMD:C_0603_1608Metric"
 			(at 63.5 54.9148 0)
 			(effects
