File: hardware/teachtaire.kicad_pcb (KiCad board)
At the start: 6 copper layers, 60 x 60 mm, 83 parts, among them J1 39-29-1048, J2 ESQ-110-X-X-D, J3 Conn_Coaxial, J4 5023860570, J5 Conn_Coaxial, Q1 NMOS, Q2 IPD90P04P4L04ATMA1, Q3 PMOS, Q4 NMOS, U1 MAX-M10S, U2 STM32F072C8Tx, U3 TJA1051T/3/1J, U4 RF-LORA-868-SO, U5 LT6003HDC-TRMPBF, U6 NC7WZ07P6X, U7 NC7WZ07P6X, U8 MPM3650CGQW-P, U9 TLV75533PDRV

Commit message: ready for review the twost
Parts:
- added 3V3D: S2761-46R, footprints:HARWIN_S2761-46R, F.Cu at (177.0, 100.0)
- added 3V3RF: S2761-46R, footprints:HARWIN_S2761-46R, F.Cu at (177.0, 104.5)
- added C+: S2761-46R, footprints:HARWIN_S2761-46R, F.Cu at (168.6, 100.3)
- added C-: S2761-46R, footprints:HARWIN_S2761-46R, F.Cu at (168.5, 105.2)
- added LD0: S2761-46R, footprints:HARWIN_S2761-46R, F.Cu at (132.8, 107.9)
- added LD1: S2761-46R, footprints:HARWIN_S2761-46R, F.Cu at (135.7, 107.9)
- added LD2: S2761-46R, footprints:HARWIN_S2761-46R, F.Cu at (138.5, 107.9)
- added LD3: S2761-46R, footprints:HARWIN_S2761-46R, F.Cu at (141.4, 108.0)
- added LD4: S2761-46R, footprints:HARWIN_S2761-46R, F.Cu at (144.2, 108.0)
- added LD5: S2761-46R, footprints:HARWIN_S2761-46R, F.Cu at (147.1, 108.0)
- added VIN: S2761-46R, footprints:HARWIN_S2761-46R, F.Cu at (177.0, 96.0)
- renumbered D4 to D1, D1 to D2, D2 to D3, D3 to D4, GND1 to GND, VBCKP1 to VBCKP
Routing:
- net VBAT: track 20.8 -> 57.7 mm, vias 4 -> 5
- net +3V3RF: track 95.2 -> 123.4 mm, vias 5 -> 6
- net GND: track 74.4 -> 88.8 mm, vias 178 -> 192
- net LoRa_DIO0: track 37.8 -> 51.4 mm
- net LoRa_DIO5: track 18.9 -> 32.2 mm
- net +3V3D: track 142.1 -> 154.2 mm, vias 11 -> 12
- net LoRa_DIO1: track 44.7 -> 54.8 mm
- net LoRa_DIO3: track 42.0 -> 51.7 mm, vias 2 -> 4
- net LoRa_DIO2: track 41.2 -> 49.8 mm
- net LoRa_DIO4: track 23.6 -> 31.5 mm
- net CANo_-: track 10.7 -> 12.6 mm
- net CANo_+: track 10.5 -> 12.4 mm
- net LoRa_RESET: track 20.9 -> 21.8 mm
Other:
- board text added: "my name is Jeff"

Commit message: crimes
Parts:
- removed J5: Conn_Coaxial, Connector_Coaxial:SMA_BAT_Wireless_BWSMA-KWE-Z001
- added J6: U.FL-R-SMT-1_10_, footprints:HRS_U.FL-R-SMT-1_10_, F.Cu at (163.2, 119.8)
- renumbered 3V3D to 3V3D1, 3V3RF to 3V3RF1, C+ to CAN+1, C- to CAN-1, GND to GND1, VBCKP to VBCKP1, VIN to VIN1
Routing:
- net Net-(C21-Pad1): track 9.37 -> 8.77 mm
- net GND: vias 192 -> 188
