File: hardware/teachtaire.kicad_pcb (KiCad board)
At the start: 6 copper layers, 60 x 60 mm, 94 parts, among them J1 39-29-1048, J2 ESQ-110-X-X-D, J3 Conn_Coaxial, J4 5023860570, J6 U.FL-R-SMT-1_10_, Q1 NMOS, Q2 IPD90P04P4L04ATMA1, Q3 PMOS, Q4 NMOS, U1 MAX-M10S, U2 STM32F072C8Tx, U3 TJA1051T/3/1J, U4 RF-LORA-868-SO, U5 LT6003HDC-TRMPBF, U6 NC7WZ07P6X, U7 NC7WZ07P6X, U8 MPM3650CGQW-P, U9 TLV75533PDRV

Commit message: ready 2 order
Parts:
- moved C15 0.14 mm to (155.4, 102.7)
- moved C16 0.14 mm to (156.4, 102.7)

Commit message: hardware done
Parts:
- removed D1: BAT54J, Diode_SMD:D_SOD-323F
- added D5: 1N4148W, Diode_SMD:D_SOD-123, F.Cu at (136.5, 117.2)
- added G***: LOGO, LOGO, F.Cu at (172.8, 120.2)
- C12, C15, C20, C22, C25, C26, C27, C29, C30, C31, C37: footprint Capacitor_SMD:C_0402_1005Metric -> Capacitor_SMD:C_0603_1608Metric
- R2: value R -> 1KΩ
- moved C32 6.09 mm to (165.7, 81.8), turned to 0 degrees
- moved C34 3.39 mm to (165.7, 82.8), turned to 180 degrees
- moved C37 2.80 mm to (166.2, 86.2), turned to 0 degrees
- moved C24 2.62 mm to (166.1, 67.9), turned to 180 degrees
- moved C16 2.12 mm to (154.2, 102.7)
- moved C12 0.80 mm to (168.1, 88.3)
- moved C27 0.77 mm to (162.6, 76.8)
- moved C25 0.70 mm to (163.7, 68.1)
- moved C31 0.65 mm to (162.6, 81.1)
- moved R6 0.42 mm to (157.1, 115.9)
- moved U3 0.39 mm to (160.1, 102.6)
- moved R5 0.37 mm to (166.0, 104.0)
- moved D4 0.36 mm to (169.0, 102.7)
- moved R4 0.35 mm to (166.0, 101.5)
- moved C22 0.35 mm to (156.9, 117.6)
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- renumbered 3V3D1 to 3V3D, 3V3RF1 to 3V3RF, CAN+1 to C+, CAN-1 to C-, GND1 to GND, VIN1 to VBAT, VBCKP1 to VBCKP
Routing:
- net +3V3D: track 154.2 -> 160.1 mm
- net GND: track 88.8 -> 91.2 mm, vias 188 -> 186
- net VBAT: track 57.7 -> 59.9 mm
- net 5VLOGIC: track 53.5 -> 54.8 mm
- net Net-(U8-VCC): track 11.5 -> 12.9 mm
- net +3V3RF: track 123.4 -> 124.7 mm
- net Net-(C20-Pad1): track 2.08 -> 3.13 mm
- net Net-(D5-A): track 3.87 -> 3.07 mm
- net CAN_-: track 17.1 -> 17.8 mm
- net CANo_-: track 12.6 -> 13.2 mm
